File: usb-uart-plug/usb-uart-plug.kicad_pcb (KiCad board)
At the start: 4 copper layers, 34.4 x 12.7 mm, 22 parts, among them J1 USB_C_Receptacle_USB2.0_14P, J10 GND, J2 UART_VIO, J3 UART_RX, J4 +5V, J5 UART_TX, J6 CC1, J7 USB_D+, J8 USB_D-, J9 CC2, U1 CH334R, U2 CP2102N-Axx-xQFN24, Y1 12MHz

Commit message: Adjust silkscreen text
Parts:
- J6: value CC1 -> USB_CC1
- J9: value CC2 -> USB_CC2
Changed lines of the file:
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@@
 			)
 		)
-		(property "Value" "CC2"
+		(property "Value" "USB_CC2"
 			(at 1.016 0 0)
 			(layer "B.SilkS")
@@
 			)
 		)
-		(property "Value" "CC1"
+		(property "Value" "USB_CC1"
 			(at 1.016 0 0)
 			(layer "B.SilkS")

Commit message: Add silkscreen text
Other:
- board text added: "JLCJLCJLCJLC"
- board text added: "USB-Uart Splitter v1"
- board text added: "by Finomnis"
Changed lines of the file:
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@@
 		(layer "Edge.Cuts")
+	)
+	(gr_text "USB-Uart\nSplitter v1"
+		(at 140.716 74.676 0)
+		(layer "B.SilkS")
+		(effects
+			(font
+				(size 1 1)
+				(thickness 0.25)
+				(bold yes)
+			)
+			(justify left bottom mirror)
+		)
+	)
+	(gr_text "JLCJLCJLCJLC"
+		(at 133.096 82.296 0)
+		(layer "B.SilkS")
+		(effects
+			(font
+				(size 0.8 0.8)
+				(thickness 0.15)
+				(bold yes)
+			)
+			(justify left bottom mirror)
+		)
+	)
+	(gr_text "by Finomnis"
+		(at 140.208 78.486 -0)
+		(layer "B.SilkS")
+		(effects
+			(font
+				(size 0.8 0.8)
+				(thickness 0.15)
+				(bold yes)
+			)
+			(justify left bottom mirror)
+		)
 	)
 	(gr_text "Stackup: JLC04161H-3313"
